Commit message: upgrade meshes with high res models from jhu-dvrk/instrument-cad

File: surrol/assets/psm/psm.urdf (robot description, URDF)
Before this commit: robot psm, 17 links, 16 joints
Links:
- link psm_tool_gripper1_link: geometry collision box size=0.0014 0.0102 0.0018; visual mesh filename=meshes/visual/gripper_right.obj
- link psm_tool_gripper2_link: geometry collision box size=0.0014 0.0102 0.0018; visual mesh filename=meshes/visual/gripper_left.obj
- link psm_tool_pitch_link: geometry collision mesh filename=meshes/visual/tool_pitch_link.OBJ; visual mesh filename=meshes/visual/tool_pitch_link.OBJ
